Commit message: Updated joint limits

File: ros/src/ball_balancer/urdf/ball_balancer.urdf (robot description, URDF)
Before this commit: robot ball_balancer, 7 links, 6 joints
Joints:
- joint servo_arm_1_joint: limit lower=0 upper=1.57 effort=1.9 velocity=5.5 -> lower=-1.57 upper=0.0 effort=1.9 velocity=5.5
- joint servo_arm_2_joint: limit lower=0 upper=1.57 effort=1.9 velocity=5.5 -> lower=-1.57 upper=0.0 effort=1.9 velocity=5.5
- joint servo_arm_3_joint: limit lower=0 upper=1.57 effort=1.9 velocity=5.5 -> lower=-1.57 upper=0.0 effort=1.9 velocity=5.5
- joint table_arm_1_joint: limit lower=-1.57 upper=0 effort=1.9 velocity=5.5 -> lower=-3.14 upper=0 effort=1.9 velocity=5.5
- joint table_arm_2_joint: limit lower=-1.57 upper=0 effort=1.9 velocity=5.5 -> lower=-3.14 upper=0 effort=1.9 velocity=5.5
- joint table_arm_3_joint: limit lower=-1.57 upper=0 effort=1.9 velocity=5.5 -> lower=-3.14 upper=0 effort=1.9 velocity=5.5

Commit message: fixed table magnet tf

File: ros/src/ball_balancer/urdf/ball_balancer.urdf (robot description, URDF)
Before this commit: robot ball_balancer, 10 links, 9 joints
Links:
- link table_arm_1_ball_link: mass 0.00256322375311019 -> None; geometry 
- link table_arm_2_ball_link: mass 0.00256321394494201 -> None; geometry 
- link table_arm_3_ball_link: mass 0.00256319746004798 -> None; geometry 
Joints:
- joint servo_arm_1_joint: limit lower=-1.57 upper=0 effort=1.9 velocity=5.5 -> lower=-1.57 upper=0.0 effort=1.9 velocity=5.5
- joint servo_arm_2_joint: limit lower=-1.57 upper=0 effort=1.9 velocity=5.5 -> lower=-1.57 upper=0.0 effort=1.9 velocity=5.5
- joint servo_arm_3_joint: limit lower=-1.57 upper=0 effort=1.9 velocity=5.5 -> lower=-1.57 upper=0.0 effort=1.9 velocity=5.5
- joint table_arm_1_ball_joint: axis 0 0 0 -> (none)
- joint table_arm_2_ball_joint: axis 0 0 0 -> (none)
- joint table_arm_3_ball_joint: axis 0 0 0 -> (none)

File: ros/src/ball_balancer_table/urdf/ball_balancer_table.urdf (robot description, URDF)
Before this commit: robot ball_balancer_table, 4 links, 3 joints
Links:
- link table_magnet_1_link: mass 0.113623772682042 -> None; geometry 
- link table_magnet_2_link: mass 0.113623772682042 -> None; geometry 
- link table_magnet_3_link: mass 0.113623772682042 -> None; geometry 
Joints:
- joint table_magnet_1_joint: origin xyz=0 -0.075 0.0005 rpy=0 0 3.1416 -> xyz=0 -0.075 -0.0045 rpy=0 0 3.1416
- joint table_magnet_2_joint: origin xyz=0.064952 0.0375 0.0005 rpy=0 0 3.1416 -> xyz=0.064952 0.0375 -0.0045 rpy=0 0 3.1416
- joint table_magnet_3_joint: origin xyz=-0.064952 0.0375 0.0005 rpy=0 0 3.1416 -> xyz=-0.064952 0.0375 -0.0045 rpy=0 0 3.1416

Commit message: Updated model again

File: ros/src/ball_balancer/urdf/ball_balancer.urdf (robot description, URDF)
Before this commit: robot ball_balancer, 7 links, 6 joints
Links:
- link servo_arm_1_link: mass 0.0030998 -> 0.00309980999161893
- link servo_arm_2_link: mass 0.0030998 -> 0.00309980999161893
- link servo_arm_3_link: mass 0 -> 0.00309980999161893
- link table_arm_2_link: mass 0.0025632 -> 0.00256321394494201
Joints:
- joint servo_arm_1_joint: origin xyz=-0.0073 -0.065736 0.03755 rpy=0 0 0 -> xyz=-0.065736 0.0073 0.03505 rpy=0 0 -1.5708
- joint servo_arm_2_joint: origin xyz=0.060579 0.026546 0.03755 rpy=0 0 2.0944 -> xyz=0.026546 -0.060579 0.03505 rpy=0 0 0.5236
- joint servo_arm_3_joint: origin xyz=-0.053279 0.03919 0.03755 rpy=0 0 -2.0944 -> xyz=0.03919 0.053279 0.03505 rpy=0 0 2.618

Commit message: Updated tf for model, added table urdf

File: ros/src/ball_balancer/urdf/ball_balancer.urdf (robot description, URDF)
Before this commit: robot ball_balancer, 7 links, 6 joints
Links:
- added link table_arm_1_ball_link, mass 0.00256322375311019; collision mesh filename=package://ball_balancer/meshes/table_arm_1_ball_link.STL; visual mesh filename=package://ball_balancer/meshes/table_arm_1_ball_link.STL
- added link table_arm_2_ball_link, mass 0.00256321394494201; collision mesh filename=package://ball_balancer/meshes/table_arm_2_ball_link.STL; visual mesh filename=package://ball_balancer/meshes/table_arm_2_ball_link.STL
- added link table_arm_3_ball_link, mass 0.00256319746004798; collision mesh filename=package://ball_balancer/meshes/table_arm_3_ball_link.STL; visual mesh filename=package://ball_balancer/meshes/table_arm_3_ball_link.STL
Joints:
- added joint table_arm_1_ball_joint: type fixed, parent table_arm_1_link, child table_arm_1_ball_link, origin xyz=0.00275 -0.054791 0 rpy=0 0 0, axis 0 0 0
- added joint table_arm_2_ball_joint: type fixed, parent table_arm_2_link, child table_arm_2_ball_link, origin xyz=0.00275 -0.054791 0 rpy=0 0 0, axis 0 0 0
- added joint table_arm_3_ball_joint: type fixed, parent table_arm_3_link, child table_arm_3_ball_link, origin xyz=0.00275 -0.054791 0 rpy=0 0 0, axis 0 0 0
- joint servo_arm_1_joint: limit lower=-1.57 upper=0.0 effort=1.9 velocity=5.5 -> lower=-1.57 upper=0 effort=1.9 velocity=5.5
- joint servo_arm_2_joint: limit lower=-1.57 upper=0.0 effort=1.9 velocity=5.5 -> lower=-1.57 upper=0 effort=1.9 velocity=5.5
- joint servo_arm_3_joint: limit lower=-1.57 upper=0.0 effort=1.9 velocity=5.5 -> lower=-1.57 upper=0 effort=1.9 velocity=5.5

Commit message: robot now in isaac

File: ros/src/ball_balancer/urdf/ball_balancer.urdf (robot description, URDF)
Before this commit: robot ball_balancer, 10 links, 9 joints
Links:
- removed link base_link
- removed link servo_arm_1_link
- removed link servo_arm_2_link
- removed link servo_arm_3_link
- removed link table_arm_1_ball_link
- removed link table_arm_1_link
- removed link table_arm_2_ball_link
- removed link table_arm_2_link
- removed link table_arm_3_ball_link
- removed link table_arm_3_link
- added link robot_base_link, mass 0.25395; collision mesh filename=package://ball_balancer2/meshes/base_link.STL; visual mesh filename=package://ball_balancer2/meshes/base_link.STL
- added link servo_arm_1, mass 0.0030998; collision mesh filename=package://ball_balancer2/meshes/servo_arm.STL; visual mesh filename=package://ball_balancer2/meshes/servo_arm.STL
- added link servo_arm_2, mass 0.00309980999161893; collision mesh filename=package://ball_balancer2/meshes/servo_arm.STL; visual mesh filename=package://ball_balancer2/meshes/servo_arm.STL
- added link servo_arm_3, mass 0.00309980999161893; collision mesh filename=package://ball_balancer2/meshes/servo_arm.STL; visual mesh filename=package://ball_balancer2/meshes/servo_arm.STL
- added link table_arm_1, mass 0.0025632; collision mesh filename=package://ball_balancer2/meshes/table_arm.STL; visual mesh filename=package://ball_balancer2/meshes/table_arm.STL
- added link table_arm_1_ball
- added link table_arm_2, mass 0.00256321315526102; collision mesh filename=package://ball_balancer2/meshes/table_arm.STL; visual mesh filename=package://ball_balancer2/meshes/table_arm.STL
- added link table_arm_2_ball
- added link table_arm_3, mass 0.00256319659543894; collision mesh filename=package://ball_balancer2/meshes/table_arm.STL; visual mesh filename=package://ball_balancer2/meshes/table_arm.STL
- added link table_arm_3_ball
- added link table_link, mass 0.113623772682042; collision mesh filename=package://ball_balancer2/meshes/table.STL; visual mesh filename=package://ball_balancer2/meshes/table.STL
- added link table_magnet_1_link
- added link table_magnet_2_link
- added link table_magnet_3_link
- added link world
Joints:
- removed joint servo_arm_1_joint
- removed joint servo_arm_2_joint
- removed joint servo_arm_3_joint
- removed joint table_arm_1_joint
- removed joint table_arm_2_joint
- removed joint table_arm_3_joint
- added joint robot_to_table_floating: type fixed, parent robot_base_link, child table_link, origin xyz=0 0 0.0665733158 rpy=0 0 0
- added joint servo_arm_1_revolute: type revolute, parent robot_base_link, child servo_arm_1, origin xyz=-0.0073 -0.065736 0.03755 rpy=0 0 0, axis -1 0 0, limit lower=-1.57 upper=0 effort=1.9 velocity=5.5
- added joint servo_arm_2_revolute: type revolute, parent robot_base_link, child servo_arm_2, origin xyz=0.060579 0.026546 0.03755 rpy=-0.010265 0 2.0944, axis -1 0 0, limit lower=-1.57 upper=0 effort=1.9 velocity=5.5
- added joint servo_arm_3_revolute: type revolute, parent robot_base_link, child servo_arm_3, origin xyz=-0.053279 0.03919 0.03755 rpy=-0.010265 0 -2.0944, axis -1 0 0, limit lower=-1.57 upper=0 effort=1.9 velocity=5.5
- added joint table_arm_1_revolute: type revolute, parent servo_arm_1, child table_arm_1, origin xyz=0.00455 0.039365 0 rpy=-0.47144 0 0, axis 1 0 0, limit lower=-3.14 upper=0 effort=1.9 velocity=5.5
- added joint table_arm_2_revolute: type revolute, parent servo_arm_2, child table_arm_2, origin xyz=0.00455 0.039365 0 rpy=-0.46126 0 0, axis 1 0 0, limit lower=-3.14 upper=0 effort=1.9 velocity=5.5
- added joint table_arm_3_revolute: type revolute, parent servo_arm_3, child table_arm_3, origin xyz=0.00455 0.039365 0 rpy=-0.46126 0 0, axis 1 0 0, limit lower=-3.14 upper=0 effort=1.9 velocity=5.5
- added joint table_magnet_1_joint: type fixed, parent table_link, child table_magnet_1_link, origin xyz=0 -0.075 -0.0045 rpy=0 0 3.1416
- added joint table_magnet_2_joint: type fixed, parent table_link, child table_magnet_2_link, origin xyz=0.064952 0.0375 -0.0045 rpy=0 0 3.1416
- added joint table_magnet_3_joint: type fixed, parent table_link, child table_magnet_3_link, origin xyz=-0.064952 0.0375 -0.0045 rpy=0 0 3.1416
- added joint world_to_robot_base: type fixed, parent world, child robot_base_link, origin xyz=0 0 0 rpy=0 0 0
- joint table_arm_1_ball_joint: child table_arm_1_ball_link -> table_arm_1_ball; origin xyz=0.00275 -0.054791 0 rpy=0 0 0 -> xyz=0.00275 -0.054583 0 rpy=0 0 0; parent table_arm_1_link -> table_arm_1
- joint table_arm_2_ball_joint: child table_arm_2_ball_link -> table_arm_2_ball; origin xyz=0.00275 -0.054791 0 rpy=0 0 0 -> xyz=0.00275 -0.054583 0 rpy=0 0 0; parent table_arm_2_link -> table_arm_2
- joint table_arm_3_ball_joint: child table_arm_3_ball_link -> table_arm_3_ball; origin xyz=0.00275 -0.054791 0 rpy=0 0 0 -> xyz=0.00275 -0.054583 0 rpy=0 0 0; parent table_arm_3_link -> table_arm_3

Commit message: Training skeleton ready

File: ros/src/ball_balancer/urdf/ball_balancer.urdf (robot description, URDF)
Before this commit: robot ball_balancer_system, 15 links, 14 joints
Links:
- removed link robot_base_link
- removed link servo_arm_1
- removed link servo_arm_2
- removed link servo_arm_3
- removed link table_arm_1
- removed link table_arm_1_ball
- removed link table_arm_2
- removed link table_arm_2_ball
- removed link table_arm_3
- removed link table_arm_3_ball
- removed link table_link
- added link Magnet_1, mass 0.511178872279149; collision mesh filename=package://ball_balancer/meshes/Magnet_1.STL; visual mesh filename=package://ball_balancer/meshes/Magnet_1.STL
- added link Magnet_2, mass 0.511178872279149; collision mesh filename=package://ball_balancer/meshes/Magnet_2.STL; visual mesh filename=package://ball_balancer/meshes/Magnet_2.STL
- added link Magnet_3, mass 0.511178872279149; collision mesh filename=package://ball_balancer/meshes/Magnet_3.STL; visual mesh filename=package://ball_balancer/meshes/Magnet_3.STL
- added link Servo_arm_1, mass 0.00867785481542915; collision mesh filename=package://ball_balancer/meshes/Servo_arm_1.STL; visual mesh filename=package://ball_balancer/meshes/Servo_arm_1.STL
- added link Servo_arm_2, mass 0.00867785481542916; collision mesh filename=package://ball_balancer/meshes/Servo_arm_2.STL; visual mesh filename=package://ball_balancer/meshes/Servo_arm_2.STL
- added link Servo_arm_3, mass 0.00867785481542916; collision mesh filename=package://ball_balancer/meshes/Servo_arm_3.STL; visual mesh filename=package://ball_balancer/meshes/Servo_arm_3.STL
- added link Table, mass 0.113623772682042; collision mesh filename=package://ball_balancer/meshes/Table.STL; visual mesh filename=package://ball_balancer/meshes/Table.STL
- added link Table_arm_1, mass 0.003906747783009; collision mesh filename=package://ball_balancer/meshes/Table_arm_1.STL; visual mesh filename=package://ball_balancer/meshes/Table_arm_1.STL
- added link Table_arm_1_ball
- added link Table_arm_2, mass 0.00390674778300901; collision mesh filename=package://ball_balancer/meshes/Table_arm_2.STL; visual mesh filename=package://ball_balancer/meshes/Table_arm_2.STL
- added link Table_arm_2_ball
- added link Table_arm_3, mass 0.003906747783009; collision mesh filename=package://ball_balancer/meshes/Table_arm_3.STL; visual mesh filename=package://ball_balancer/meshes/Table_arm_3.STL
- added link Table_arm_3_ball
- added link base_link, mass 0.330312516893083; collision mesh filename=package://ball_balancer/meshes/base_link.STL; visual mesh filename=package://ball_balancer/meshes/base_link.STL
Joints:
- removed joint robot_to_table_floating
- removed joint servo_arm_1_revolute
- removed joint servo_arm_2_revolute
- removed joint servo_arm_3_revolute
- removed joint table_arm_1_ball_joint
- removed joint table_arm_1_revolute
- removed joint table_arm_2_ball_joint
- removed joint table_arm_2_revolute
- removed joint table_arm_3_ball_joint
- removed joint table_arm_3_revolute
- removed joint world_to_robot_base
- added joint Magnet_1_mesh_joint: type fixed, parent table_magnet_1_link, child Magnet_1, origin xyz=0 0 0 rpy=0 0 0
- added joint Magnet_2_mesh_joint: type fixed, parent table_magnet_2_link, child Magnet_2, origin xyz=0 0 0 rpy=0 0 0
- added joint Magnet_3_mesh_joint: type fixed, parent table_magnet_3_link, child Magnet_3, origin xyz=0 0 0 rpy=0 0 0
- added joint Servo_arm_1_revolute: type revolute, parent base_link, child Servo_arm_1, origin xyz=0.063196 -0.0049738 0.07505 rpy=0 0 1.5708, axis -1 0 0, limit lower=0 upper=0 effort=0 velocity=0
- added joint Servo_arm_2_revolute: type revolute, parent base_link, child Servo_arm_2, origin xyz=-0.032304 -0.060111 0.07505 rpy=0 0 -0.5236, axis -1 0 0, limit lower=0 upper=0 effort=0 velocity=0
- added joint Servo_arm_3_revolute: type revolute, parent base_link, child Servo_arm_3, origin xyz=-0.032304 0.050163 0.07505 rpy=0 0 -2.618, axis -1 0 0, limit lower=0 upper=0 effort=0 velocity=0
- added joint Table_arm_1_ball_joint: type fixed, parent Table_arm_1, child Table_arm_1_ball, origin xyz=0 -0.053793 0 rpy=0 0 0
- added joint Table_arm_1_revolute: type revolute, parent Servo_arm_1, child Table_arm_1, origin xyz=0 0.039365 0 rpy=-0.39093 0 0, axis -1 0 0, limit lower=0 upper=0 effort=0 velocity=0
- added joint Table_arm_2_ball_joint: type fixed, parent Table_arm_2, child Table_arm_2_ball, origin xyz=0 -0.053793 0 rpy=0 0 0
- added joint Table_arm_2_revolute: type revolute, parent Servo_arm_2, child Table_arm_2, origin xyz=0 0.039365 0 rpy=-0.39093 0 0, axis 1 0 0, limit lower=0 upper=0 effort=0 velocity=0
- added joint Table_arm_3_ball_joint: type fixed, parent Table_arm_3, child Table_arm_3_ball, origin xyz=0 -0.053793 0 rpy=0 0 0
- added joint Table_arm_3_revolute: type revolute, parent Servo_arm_3, child Table_arm_3, origin xyz=0 0.039365 0 rpy=-0.39093 0 0, axis -1 0 0, limit lower=0 upper=0 effort=0 velocity=0
- added joint Table_joint: type fixed, parent base_link, child Table, origin xyz=-0.00047047 -0.0049738 0.10505 rpy=0 0 0
- added joint world_to_base_link: type fixed, parent world, child base_link, origin xyz=0 0 0 rpy=0 0 0
- joint table_magnet_1_joint: origin xyz=0 -0.075 -0.0045 rpy=0 0 3.1416 -> xyz=0.074036 0 -0.0095 rpy=0 0 0; parent table_link -> Table
- joint table_magnet_2_joint: origin xyz=0.064952 0.0375 -0.0045 rpy=0 0 3.1416 -> xyz=-0.037018 -0.064117 -0.0095 rpy=0 0 0; parent table_link -> Table
- joint table_magnet_3_joint: origin xyz=-0.064952 0.0375 -0.0045 rpy=0 0 3.1416 -> xyz=-0.037018 0.064117 -0.0095 rpy=0 0 0; parent table_link -> Table
